File: 8-DI-ESP32-PCB.sch (KiCad schematic (older format))
At the start: 67 parts, among them J1 Conn_01x03_Male, J10 Screw_Terminal_01x02, J11 PROGRAM CONN., J2 Conn_01x03_Male, J3 Conn_01x03_Male, J4 Conn_01x03_Male, J5 Conn_01x03_Male, J6 Conn_01x03_Male, J7 Conn_01x03_Male, J8 Conn_01x03_Male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

Commit message: clean-up temp. files
Parts:
- U3: symbol 8-DI-ESP32-PCB-rescue:ESP32-WROVER-IE-ESP32-WROVER-IE -> ESP32-WROVER-IE:ESP32-WROVER-IE
Changed lines of the file:
@@
 $EndComp
 $Comp
-L 8-DI-ESP32-PCB-rescue:ESP32-WROVER-IE-ESP32-WROVER-IE U3
+L ESP32-WROVER-IE:ESP32-WROVER-IE U3
 U 1 1 5F8D92F8
 P 5300 1200
